Commit message: First batch

File: bundle/deepracer_simulation_environment/share/deepracer_simulation_environment/urdf/confetti/macros.xacro (robot description, xacro)
@@ -53,4 +53,10 @@
   <geometry>
     <mesh filename="package://deepracer_simulation_environment/meshes/confetti/top_cover_two_cameras.STL"/>
+  </geometry>
+</xacro:macro>
+<xacro:macro name="f1_geometry"  params="body_shell_type">
+  <origin xyz="0.12 0 -0.05" rpy="0 0 0" />
+  <geometry>
+    <mesh filename="package://deepracer_simulation_environment/meshes/f1/${body_shell_type}.dae"/>
   </geometry>
 </xacro:macro>

File: bundle/deepracer_simulation_environment/share/deepracer_simulation_environment/urdf/confetti/racecar.xacro (robot description, xacro)
@@ -20,5 +20,6 @@
   <xacro:arg name="disable_gazebo_sensors" default="false" />
   <xacro:arg name="single_camera_racecar_body" default="true" />
-  <xacro:arg name="car_color" default="Black" />
+  <xacro:arg name="body_shell_type" default="deepracer" />
+  <xacro:property name="body_shell_type_val" value="$(arg body_shell_type)" />
   <!-- Add chassis and it's inertia link -->
   <link name="base_link" />
@@ -187,8 +188,13 @@
   <xacro:unless value="$(arg single_camera_racecar_body)">
   <link
-    name="top_cover_lidar_two_cameras_link">
+    name="car_body_link_v2">
     <xacro:if value="$(arg include_lidar_sensor)">
       <visual>
-        <xacro:top_cover_lidar_two_cameras_geometry />
+        <xacro:unless value="${'f1' in body_shell_type_val}">
+          <xacro:top_cover_lidar_two_cameras_geometry />
+        </xacro:unless>
+        <xacro:if value="${'f1' in body_shell_type_val}">
+          <xacro:f1_geometry body_shell_type="$(arg body_shell_type)"/>
+        </xacro:if>
       </visual>
       <collision>
@@ -198,5 +204,10 @@
     <xacro:unless value="$(arg include_lidar_sensor)">
       <visual>
-        <xacro:top_cover_two_cameras_geometry />
+        <xacro:unless value="${'f1' in body_shell_type_val}">
+          <xacro:top_cover_two_cameras_geometry />
+        </xacro:unless>
+        <xacro:if value="${'f1' in body_shell_type_val}">
+          <xacro:f1_geometry body_shell_type="$(arg body_shell_type)"/>
+        </xacro:if>
       </visual>
       <collision>
@@ -205,9 +216,9 @@
     </xacro:unless>
   </link>
-  <xacro:configure_collide_bitmask link_name="top_cover_lidar_two_cameras_link" bitmask="$(arg racecar_bitmask)" />
-  <joint name="top_cover_lidar_two_cameras_link_joint" type="fixed">
+  <xacro:configure_collide_bitmask link_name="car_body_link_v2" bitmask="$(arg racecar_bitmask)" />
+  <joint name="car_body_link_joint" type="fixed">
     <origin xyz="-0.02 0 0.02" rpy="0 0 0"/>
     <parent link="chassis"/>
-    <child link="top_cover_lidar_two_cameras_link"/>
+    <child link="car_body_link_v2"/>
     <axis xyz="0 0 1" />
   </joint>
@@ -217,11 +228,16 @@
       <visual>
         <!-- Lowering the car body for the bot car-->
-        <xacro:unless value="$(arg disable_gazebo_sensors)">
-          <origin xyz="0.1 0 0" rpy="0 0 3.1415926535898" />
+        <xacro:unless value="${'f1' in body_shell_type_val}">
+          <xacro:unless value="$(arg disable_gazebo_sensors)">
+            <origin xyz="0.1 0 0" rpy="0 0 3.1415926535898" />
+          </xacro:unless>
+          <xacro:if value="$(arg disable_gazebo_sensors)">
+            <origin xyz="0.09 0 -0.02" rpy="0 0 3.1415926535898" />
+          </xacro:if>
+          <xacro:body_visual_geometry />
         </xacro:unless>
-        <xacro:if value="$(arg disable_gazebo_sensors)">
-          <origin xyz="0.09 0 -0.02" rpy="0 0 3.1415926535898" />
+        <xacro:if value="${'f1' in body_shell_type_val}">
+          <xacro:f1_geometry body_shell_type="$(arg body_shell_type)"/>
         </xacro:if>
-        <xacro:body_visual_geometry />
       </visual>
       <collision>

File: bundle/deepracer_simulation_environment/share/deepracer_simulation_environment/urdf/mit/macros.xacro (robot description, xacro)
@@ -35,4 +35,10 @@
   <geometry>
     <mesh filename="package://deepracer_simulation_environment/meshes/mit/top_cover.STL"/>
+  </geometry>
+</xacro:macro>
+<xacro:macro name="f1_geometry"  params="body_shell_type">
+  <origin xyz="0.12 0 -0.05" rpy="0 0 0" />
+  <geometry>
+    <mesh filename="package://deepracer_simulation_environment/meshes/f1/${body_shell_type}.dae"/>
   </geometry>
 </xacro:macro>

File: bundle/deepracer_simulation_environment/share/deepracer_simulation_environment/urdf/mit/racecar.xacro (robot description, xacro)
@@ -6,5 +6,6 @@
   <xacro:arg name="include_second_camera" default="false" />
   <xacro:arg name="include_lidar_sensor" default="false" />
-  <xacro:arg name="car_color" default="Black" />
+  <xacro:arg name="body_shell_type" default="deepracer" />
+  <xacro:property name="body_shell_type_val" value="$(arg body_shell_type)" />
   <!-- Add chassis and it's inertia link -->
   <link name="base_link" />
@@ -175,5 +176,10 @@
   <link name="top_cover_link">
     <visual>
-      <xacro:top_cover_geometry />
+      <xacro:unless value="${'f1' in body_shell_type_val}">
+        <xacro:top_cover_geometry />
+      </xacro:unless>
+      <xacro:if value="${'f1' in body_shell_type_val}">
+        <xacro:f1_geometry body_shell_type="$(arg body_shell_type)"/>
+      </xacro:if>
     </visual>
     <collision>
