Commit message: Initial batch

File: bundle/deepracer_simulation_environment/share/deepracer_simulation_environment/urdf/confetti/racecar.xacro (robot description, xacro)
@@ -19,5 +19,4 @@
   <!-- Racecar body -->
   <xacro:arg name="disable_gazebo_sensors" default="false" />
-  <xacro:arg name="single_camera_racecar_body" default="true" />
   <xacro:arg name="body_shell_type" default="deepracer" />
   <xacro:property name="body_shell_type_val" value="$(arg body_shell_type)" />
@@ -185,8 +184,13 @@
   </joint>
   <xacro:wheel_transmission name="right_front_wheel" />
-   <!-- The bot cars will have older confetti models. Since we dont have the .dae files -->
-  <xacro:unless value="$(arg single_camera_racecar_body)">
+  <!-- config f1 shell -->
+  <xacro:if value="${'f1' in body_shell_type_val}">
+    <xacro:property name="body_link_name" value="f1_body_link" />
+  </xacro:if>
+  <xacro:unless value="${'f1' in body_shell_type_val}">
+    <xacro:property name="body_link_name" value="car_body_link_v2" />
+  </xacro:unless>
   <link
-    name="car_body_link_v2">
+    name="${body_link_name}">
     <xacro:if value="$(arg include_lidar_sensor)">
       <visual>
@@ -216,47 +220,11 @@
     </xacro:unless>
   </link>
-  <xacro:configure_collide_bitmask link_name="car_body_link_v2" bitmask="$(arg racecar_bitmask)" />
+  <xacro:configure_collide_bitmask link_name="${body_link_name}" bitmask="$(arg racecar_bitmask)" />
   <joint name="car_body_link_joint" type="fixed">
     <origin xyz="-0.02 0 0.02" rpy="0 0 0"/>
     <parent link="chassis"/>
-    <child link="car_body_link_v2"/>
+    <child link="${body_link_name}"/>
     <axis xyz="0 0 1" />
   </joint>
-  </xacro:unless>
-  <xacro:if value="$(arg single_camera_racecar_body)">
-    <link name="car_body_link">
-      <visual>
-        <!-- Lowering the car body for the bot car-->
-        <xacro:unless value="${'f1' in body_shell_type_val}">
-          <xacro:unless value="$(arg disable_gazebo_sensors)">
-            <origin xyz="0.1 0 0" rpy="0 0 3.1415926535898" />
-          </xacro:unless>
-          <xacro:if value="$(arg disable_gazebo_sensors)">
-            <origin xyz="0.09 0 -0.02" rpy="0 0 3.1415926535898" />
-          </xacro:if>
-          <xacro:body_visual_geometry />
-        </xacro:unless>
-        <xacro:if value="${'f1' in body_shell_type_val}">
-          <xacro:f1_geometry body_shell_type="$(arg body_shell_type)"/>
-        </xacro:if>
-      </visual>
-      <collision>
-        <xacro:unless value="$(arg disable_gazebo_sensors)">
-          <origin xyz="0.1 0 0" rpy="0 0 3.1415926535898" />
-        </xacro:unless>
-        <xacro:if value="$(arg disable_gazebo_sensors)">
-          <origin xyz="0.09 0 -0.02" rpy="0 0 3.1415926535898" />
-        </xacro:if>
-        <xacro:body_visual_geometry />
-      </collision>
-    </link>
-    <xacro:configure_collide_bitmask link_name="car_body_link" bitmask="$(arg racecar_bitmask)" />
-    <joint name="car_body_link_joint" type="fixed">
-      <origin xyz="0 0 0.10368" rpy="0 0 0"/>
-      <parent link="chassis"/>
-      <child link="car_body_link"/>
-      <axis xyz="0 0 1" />
-    </joint>
-  </xacro:if>
   <xacro:unless value="$(arg include_second_camera)">
     <xacro:camera_module suffix="" y="0" />

File: bundle/deepracer_simulation_environment/share/deepracer_simulation_environment/urdf/mit/racecar.xacro (robot description, xacro)
@@ -173,6 +173,12 @@
     <!-- <limit lower="0.0" upper="0.0" effort="0.0" velocity="0.0" /> -->
   </joint>
-   <!-- The bot cars will have older confetti models. Since we dont have the .dae files -->
-  <link name="top_cover_link">
+  <!-- config f1 shell -->
+  <xacro:if value="${'f1' in body_shell_type_val}">
+    <xacro:property name="body_link_name" value="f1_body_link" />
+  </xacro:if>
+  <xacro:unless value="${'f1' in body_shell_type_val}">
+    <xacro:property name="body_link_name" value="car_body_link_v1" />
+  </xacro:unless>
+  <link name="${body_link_name}">
     <visual>
       <xacro:unless value="${'f1' in body_shell_type_val}">
@@ -187,9 +193,9 @@
     </collision>
   </link>
-  <xacro:configure_collide_bitmask link_name="top_cover_link" bitmask="$(arg racecar_bitmask)" />
-  <joint name="top_cover_link_joint" type="fixed">
+  <xacro:configure_collide_bitmask link_name="${body_link_name}" bitmask="$(arg racecar_bitmask)" />
+  <joint name="car_body_link_joint" type="fixed">
     <origin xyz="-0.02 0 0.02" rpy="0 0 0"/>
     <parent link="chassis"/>
-    <child link="top_cover_link"/>
+    <child link="${body_link_name}"/>
     <axis xyz="0 0 1" />
   </joint>
