Commit message: Adding deepracer_kinematics

File: bundle/deepracer_simulation_environment/share/deepracer_simulation_environment/urdf/deepracer/deepracer_single_cam.urdf (robot description, URDF)
Before this commit: robot deepracer_single_cam, 11 links, 10 joints
Links:
- link car_body_link_v3: geometry collision mesh filename=package://deepracer_simulation_environment/meshes/deepracer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
- link left_front_wheel: geometry collision mesh filename=package://deepracer_simulation_environment/meshes/deepracer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
- link left_rear_wheel: geometry collision mesh filename=package://deepracer_simulation_environment/meshes/deepracer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
- link left_steering_hinge: geometry 
- link right_front_wheel: geometry collision mesh filename=package://deepracer_simulation_environment/meshes/deepracer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
- link right_rear_wheel: geometry collision mesh filename=package://deepracer_simulation_environment/meshes/deepracer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
- link right_steering_hinge: geometry 
- link zed_camera_link: geometry 

File: bundle/deepracer_simulation_environment/share/deepracer_simulation_environment/urdf/deepracer/deepracer_single_cam_lidar.urdf (robot description, URDF)
Before this commit: robot deepracer_single_cam_lidar, 12 links, 11 joints
Links:
- link car_body_link_v3: geometry collision mesh filename=package://deepracer_simulation_environment/meshes/deepracer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
- link laser: geometry collision mesh filename=package://deepracer_simulation_environment/meshes/deepracer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
- link left_front_wheel: geometry collision mesh filename=package://deepracer_simulation_environment/meshes/deepracer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
- link left_rear_wheel: geometry collision mesh filename=package://deepracer_simulation_environment/meshes/deepracer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
- link left_steering_hinge: geometry 
- link right_front_wheel: geometry collision mesh filename=package://deepracer_simulation_environment/meshes/deepracer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
- link right_rear_wheel: geometry collision mesh filename=package://deepracer_simulation_environment/meshes/deepracer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
- link right_steering_hinge: geometry 
- link zed_camera_link: geometry 

File: bundle/deepracer_simulation_environment/share/deepracer_simulation_environment/urdf/deepracer/deepracer_stereo_cam.urdf (robot description, URDF)
Before this commit: robot deepracer_stereo_cam, 13 links, 12 joints
Links:
- link car_body_link_v3: geometry collision mesh filename=package://deepracer_simulation_environment/meshes/deepracer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
- link left_front_wheel: geometry collision mesh filename=package://deepracer_simulation_environment/meshes/deepracer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
- link left_rear_wheel: geometry collision mesh filename=package://deepracer_simulation_environment/meshes/deepracer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
- link left_steering_hinge: geometry 
- link right_front_wheel: geometry collision mesh filename=package://deepracer_simulation_environment/meshes/deepracer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
- link right_rear_wheel: geometry collision mesh filename=package://deepracer_simulation_environment/meshes/deepracer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
- link right_steering_hinge: geometry 
- link zed_camera_link_leftcam: geometry 
- link zed_camera_link_rightcam: geometry 

File: bundle/deepracer_simulation_environment/share/deepracer_simulation_environment/urdf/deepracer/deepracer_stereo_cam_lidar.urdf (robot description, URDF)
Before this commit: robot deepracer_stereo_cam_lidar, 14 links, 13 joints
Links:
- link car_body_link_v3: geometry collision mesh filename=package://deepracer_simulation_environment/meshes/deepracer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
- link laser: geometry collision mesh filename=package://deepracer_simulation_environment/meshes/deepracer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
- link left_front_wheel: geometry collision mesh filename=package://deepracer_simulation_environment/meshes/deepracer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
- link left_rear_wheel: geometry collision mesh filename=package://deepracer_simulation_environment/meshes/deepracer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
- link left_steering_hinge: geometry 
- link right_front_wheel: geometry collision mesh filename=package://deepracer_simulation_environment/meshes/deepracer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
- link right_rear_wheel: geometry collision mesh filename=package://deepracer_simulation_environment/meshes/deepracer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
- link right_steering_hinge: geometry 
- link zed_camera_link_leftcam: geometry 
- link zed_camera_link_rightcam: geometry 
