Commit message: Merging the IMU experimental branch to latest layout

File: bundle/urdf/deepracer/deepracer_single_cam.urdf (robot description, URDF)
Before this commit: robot deepracer_single_cam, 11 links, 10 joints
Links:
- added link imu_link, mass 0
Joints:
- added joint car_imu_joint: type fixed, parent chassis, child imu_link, origin xyz=-0.0762 0 2E-05 rpy=0 0 0, axis 0 0 0

File: bundle/urdf/deepracer/deepracer_single_cam_lidar.urdf (robot description, URDF)
Before this commit: robot deepracer_single_cam_lidar, 12 links, 11 joints
Links:
- added link imu_link, mass 0
Joints:
- added joint car_imu_joint: type fixed, parent chassis, child imu_link, origin xyz=0 0 0 rpy=0 0 0, axis 0 0 0

File: bundle/urdf/deepracer/deepracer_stereo_cam.urdf (robot description, URDF)
Before this commit: robot deepracer_stereo_cam, 13 links, 12 joints
Links:
- added link imu_link, mass 0
Joints:
- added joint car_imu_joint: type fixed, parent chassis, child imu_link, origin xyz=0 0 0 rpy=0 0 0, axis 0 0 0

File: bundle/urdf/deepracer/deepracer_stereo_cam_lidar.urdf (robot description, URDF)
Before this commit: robot deepracer_stereo_cam_lidar, 14 links, 13 joints
Links:
- added link imu_link, mass 0
Joints:
- added joint car_imu_joint: type fixed, parent chassis, child imu_link, origin xyz=0 0 0 rpy=0 0 0, axis 0 0 0

File: bundle/urdf/deepracer/racecar.xacro (robot description, xacro)
@@ -9,4 +9,5 @@
   <xacro:arg name="include_second_camera" default="false" />
   <xacro:arg name="include_lidar_sensor" default="false" />
+  <xacro:arg name="include_imu_sensor" default="false" />
   <!-- lidar 360 degree - settings -->
   <xacro:arg name="lidar_360_degree_sample" default="61" />
